File: arduino-oled-shield/ProtoShield_V4.0.sch (EAGLE design)
At the start: 22 parts

Commit message: oled shield update
Parts:
- added LED1: (no value), led:LED3MM
- added R8: (no value), resistor:R-EU_0207/10
Connections:
- new net N$24: LED1.A, R8.1
- net GND: now also LED1.C
- net N$1: now also R8.2
Changed lines of the file:
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@@
 <part name="P+7" library="supply1" deviceset="VCC" device=""/>
 <part name="GND8" library="supply1" deviceset="GND" device=""/>
+<part name="LED1" library="led" deviceset="LED" device="3MM"/>
+<part name="R8" library="resistor" deviceset="R-EU_" device="0207/10"/>
+<part name="GND9" library="supply1" deviceset="GND" device=""/>
 </parts>
 <sheets>
@@
 <instance part="P+7" gate="VCC" x="167.64" y="48.26"/>
 <instance part="GND8" gate="1" x="167.64" y="27.94"/>
+<instance part="LED1" gate="G$1" x="162.56" y="83.82"/>
+<instance part="R8" gate="G$1" x="162.56" y="99.06" rot="R90"/>
+<instance part="GND9" gate="1" x="162.56" y="73.66"/>
 </instances>
 <busses>
@@
 <wire x1="200.66" y1="106.68" x2="185.42" y2="106.68" width="0.1524" layer="91"/>
 <pinref part="DIGITAL-H2" gate="A" pin="6"/>
+<wire x1="185.42" y1="106.68" x2="162.56" y2="106.68" width="0.1524" layer="91"/>
+<pinref part="R8" gate="G$1" pin="2"/>
+<wire x1="162.56" y1="106.68" x2="162.56" y2="104.14" width="0.1524" layer="91"/>
 </segment>
 </net>
@@
 <wire x1="15.24" y1="27.94" x2="17.78" y2="27.94" width="0.1524" layer="91"/>
 </segment>
+<segment>
+<pinref part="LED1" gate="G$1" pin="C"/>
+<pinref part="GND9" gate="1" pin="GND"/>
+<wire x1="162.56" y1="78.74" x2="162.56" y2="76.2" width="0.1524" layer="91"/>
+</segment>
 </net>
 <net name="VCC" class="0">
@@
 </segment>
 </net>
+<net name="N$24" class="0">
+<segment>
+<pinref part="R8" gate="G$1" pin="1"/>
+<pinref part="LED1" gate="G$1" pin="A"/>
+<wire x1="162.56" y1="93.98" x2="162.56" y2="86.36" width="0.1524" layer="91"/>
+</segment>
+</net>

Commit message: board signal clearance fix
Connections:
- net GND: now also DIGITAL-H1.7, DIGITAL-H2.7; no longer S1.P, S2.P, S2.P1
- net N$16: now also S1.P, S2.P1; no longer DIGITAL-H1.7, DIGITAL-H2.7
- net N$26: now also S3.S1; no longer S3.S
- net N$31: now also S5.S1; no longer S5.S
- net N$37: now also S5.S; no longer S5.S1
Other:
- moved on the sheet: R3, R5
Changed lines of the file:
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@@
 <classes>
 <class number="0" name="default" width="0" drill="0">
+<clearance class="0" value="0.405"/>
 </class>
 </classes>
@@
 <part name="R7" library="resistor" deviceset="R-EU_" device="0207/10"/>
 <part name="GND1" library="supply1" deviceset="GND" device=""/>
-<part name="GND2" library="supply1" deviceset="GND" device=""/>
 <part name="GND3" library="supply1" deviceset="GND" device=""/>
 <part name="GND4" library="supply1" deviceset="GND" device=""/>
@@
 <part name="R8" library="resistor" deviceset="R-EU_" device="0207/10"/>
 <part name="GND9" library="supply1" deviceset="GND" device=""/>
+<part name="GND10" library="supply1" deviceset="GND" device=""/>
 </parts>
 <sheets>
@@
 <instance part="R1" gate="G$1" x="-2.54" y="53.34" rot="R90"/>
 <instance part="R2" gate="G$1" x="15.24" y="53.34" rot="R90"/>
-<instance part="R3" gate="G$1" x="35.56" y="53.34" rot="R90"/>
+<instance part="R3" gate="G$1" x="38.1" y="53.34" rot="R90"/>
 <instance part="R4" gate="G$1" x="55.88" y="53.34" rot="R90"/>
-<instance part="R5" gate="G$1" x="76.2" y="53.34" rot="R90"/>
+<instance part="R5" gate="G$1" x="78.74" y="53.34" rot="R90"/>
 <instance part="R6" gate="G$1" x="167.64" y="134.62" rot="R90"/>
 <instance part="R7" gate="G$1" x="172.72" y="134.62" rot="R90"/>
 <instance part="GND1" gate="1" x="-2.54" y="17.78"/>
-<instance part="GND2" gate="1" x="17.78" y="17.78"/>
 <instance part="GND3" gate="1" x="38.1" y="17.78"/>
 <instance part="GND4" gate="1" x="55.88" y="17.78"/>
@@
 <instance part="P+1" gate="VCC" x="-2.54" y="66.04"/>
 <instance part="P+2" gate="VCC" x="15.24" y="66.04"/>
-<instance part="P+3" gate="VCC" x="35.56" y="66.04"/>
+<instance part="P+3" gate="VCC" x="38.1" y="66.04"/>
 <instance part="P+4" gate="VCC" x="55.88" y="66.04"/>
-<instance part="P+5" gate="VCC" x="76.2" y="66.04"/>
+<instance part="P+5" gate="VCC" x="78.74" y="66.04"/>
 <instance part="GND6" gate="1" x="91.44" y="76.2"/>
 <instance part="GND7" gate="1" x="144.78" y="99.06"/>
@@
 <instance part="R8" gate="G$1" x="162.56" y="99.06" rot="R90"/>
 <instance part="GND9" gate="1" x="162.56" y="73.66"/>
+<instance part="GND10" gate="1" x="172.72" y="96.52"/>
 </instances>
 <busses>
@@
 </segment>
 </net>
-<net name="N$16" class="0">
-<segment>
-<pinref part="DIGITAL-H1" gate="A" pin="7"/>
-<wire x1="200.66" y1="109.22" x2="185.42" y2="109.22" width="0.1524" layer="91"/>
-<pinref part="DIGITAL-H2" gate="A" pin="7"/>
-</segment>
-</net>
 <net name="N$13" class="0">
 <segment>
@@
 <net name="N$26" class="0">
 <segment>
-<pinref part="S3" gate="1" pin="S"/>
 <pinref part="R3" gate="G$1" pin="1"/>
-<wire x1="35.56" y1="38.1" x2="35.56" y2="43.18" width="0.1524" layer="91"/>
 <pinref part="U$1" gate="G$1" pin="P7"/>
-<wire x1="35.56" y1="43.18" x2="35.56" y2="48.26" width="0.1524" layer="91"/>
+<wire x1="38.1" y1="43.18" x2="38.1" y2="48.26" width="0.1524" layer="91"/>
 <wire x1="96.52" y1="101.6" x2="43.18" y2="101.6" width="0.1524" layer="91"/>
 <wire x1="43.18" y1="101.6" x2="43.18" y2="43.18" width="0.1524" layer="91"/>
-<wire x1="43.18" y1="43.18" x2="35.56" y2="43.18" width="0.1524" layer="91"/>
-<junction x="35.56" y="43.18"/>
+<wire x1="43.18" y1="43.18" x2="38.1" y2="43.18" width="0.1524" layer="91"/>
+<pinref part="S3" gate="1" pin="S1"/>
+<wire x1="38.1" y1="43.18" x2="38.1" y2="38.1" width="0.1524" layer="91"/>
 </segment>
 </net>
@@
 </segment>
 </net>
-<net name="N$31" class="0">
-<segment>
-<pinref part="S5" gate="1" pin="S"/>
-<pinref part="R5" gate="G$1" pin="1"/>
-<wire x1="76.2" y1="38.1" x2="76.2" y2="48.26" width="0.1524" layer="91"/>
-</segment>
-</net>
 <net name="N$37" class="0">
 <segment>
 <pinref part="U$1" gate="G$1" pin="P2"/>
 <wire x1="96.52" y1="114.3" x2="83.82" y2="114.3" width="0.1524" layer="91"/>
-<wire x1="83.82" y1="114.3" x2="83.82" y2="38.1" width="0.1524" layer="91"/>
-<pinref part="S5" gate="1" pin="S1"/>
-<wire x1="83.82" y1="38.1" x2="78.74" y2="38.1" width="0.1524" layer="91"/>
+<wire x1="83.82" y1="114.3" x2="83.82" y2="43.18" width="0.1524" layer="91"/>
+<pinref part="S5" gate="1" pin="S"/>
+<wire x1="76.2" y1="38.1" x2="76.2" y2="43.18" width="0.1524" layer="91"/>
+<wire x1="76.2" y1="43.18" x2="83.82" y2="43.18" width="0.1524" layer="91"/>
 </segment>
 </net>
@@
 <pinref part="GND1" gate="1" pin="GND"/>
 <wire x1="-2.54" y1="27.94" x2="-2.54" y2="20.32" width="0.1524" layer="91"/>
-<pinref part="S1" gate="1" pin="P"/>
-<wire x1="-5.08" y1="27.94" x2="-2.54" y2="27.94" width="0.1524" layer="91"/>
 </segment>
 <segment>
@@
 </segment>
 <segment>
+<pinref part="LED1" gate="G$1" pin="C"/>
+<pinref part="GND9" gate="1" pin="GND"/>
+<wire x1="162.56" y1="78.74" x2="162.56" y2="76.2" width="0.1524" layer="91"/>
+</segment>
+<segment>
+<pinref part="DIGITAL-H1" gate="A" pin="7"/>
+<wire x1="200.66" y1="109.22" x2="185.42" y2="109.22" width="0.1524" layer="91"/>
+<pinref part="DIGITAL-H2" gate="A" pin="7"/>
+<wire x1="185.42" y1="109.22" x2="177.8" y2="109.22" width="0.1524" layer="91"/>
+<wire x1="177.8" y1="109.22" x2="172.72" y2="109.22" width="0.1524" layer="91"/>
+<wire x1="172.72" y1="109.22" x2="172.72" y2="99.06" width="0.1524" layer="91"/>
+<pinref part="GND10" gate="1" pin="GND"/>
 <wire x1="200.66" y1="35.56" x2="185.42" y2="35.56" width="0.1524" layer="91"/>
 <pinref part="POWER2" gate="A" pin="6"/>
 <pinref part="POWER1" gate="A" pin="6"/>
-<wire x1="185.42" y1="35.56" x2="167.64" y2="35.56" width="0.1524" layer="91"/>
+<wire x1="185.42" y1="35.56" x2="177.8" y2="35.56" width="0.1524" layer="91"/>
+<wire x1="177.8" y1="35.56" x2="167.64" y2="35.56" width="0.1524" layer="91"/>
 <wire x1="167.64" y1="35.56" x2="167.64" y2="30.48" width="0.1524" layer="91"/>
 <pinref part="GND8" gate="1" pin="GND"/>
-</segment>
-<segment>
-<pinref part="S2" gate="1" pin="P1"/>
-<pinref part="GND2" gate="1" pin="GND"/>
-<wire x1="17.78" y1="27.94" x2="17.78" y2="20.32" width="0.1524" layer="91"/>
-<pinref part="S2" gate="1" pin="P"/>
-<wire x1="15.24" y1="27.94" x2="17.78" y2="27.94" width="0.1524" layer="91"/>
-</segment>
-<segment>
-<pinref part="LED1" gate="G$1" pin="C"/>
-<pinref part="GND9" gate="1" pin="GND"/>
-<wire x1="162.56" y1="78.74" x2="162.56" y2="76.2" width="0.1524" layer="91"/>
+<wire x1="177.8" y1="109.22" x2="177.8" y2="35.56" width="0.1524" layer="91"/>
+<junction x="177.8" y="109.22"/>
+<junction x="177.8" y="35.56"/>
 </segment>
 </net>
@@
 <pinref part="P+3" gate="VCC" pin="VCC"/>
 <pinref part="R3" gate="G$1" pin="2"/>
-<wire x1="35.56" y1="63.5" x2="35.56" y2="58.42" width="0.1524" layer="91"/>
+<wire x1="38.1" y1="63.5" x2="38.1" y2="58.42" width="0.1524" layer="91"/>
 </segment>
 <segment>
@@
 <pinref part="P+5" gate="VCC" pin="VCC"/>
 <pinref part="R5" gate="G$1" pin="2"/>
-<wire x1="76.2" y1="63.5" x2="76.2" y2="58.42" width="0.1524" layer="91"/>
+<wire x1="78.74" y1="63.5" x2="78.74" y2="58.42" width="0.1524" layer="91"/>
 </segment>
 <segment>
@@
 </segment>
 </net>
+<net name="N$16" class="0">
+<segment>
+<pinref part="S1" gate="1" pin="P"/>
+<wire x1="-5.08" y1="27.94" x2="-5.08" y2="25.4" width="0.1524" layer="91"/>
+<wire x1="-5.08" y1="25.4" x2="17.78" y2="25.4" width="0.1524" layer="91"/>
+<pinref part="S2" gate="1" pin="P1"/>
+<wire x1="17.78" y1="25.4" x2="17.78" y2="27.94" width="0.1524" layer="91"/>
+</segment>
+</net>
+<net name="N$31" class="0">
+<segment>
+<pinref part="R5" gate="G$1" pin="1"/>
+<pinref part="S5" gate="1" pin="S1"/>
+<wire x1="78.74" y1="48.26" x2="78.74" y2="38.1" width="0.1524" layer="91"/>
+</segment>
+</net>
